Commit message: Added State Interfaces
Signed-off-by: nitin2606 <nitinmaurya2606@gmail.com>

File: src/swerve_drive_description/urdf/macros.xacro (robot description, xacro)
@@ -1,32 +1,246 @@
-<?xml version="1.0"?>
-<robot xmlns:xacro="http://www.ros.org/wiki/xacro" >
-    <!-- Specify some standard inertial calculations https://en.wikipedia.org/wiki/List_of_moments_of_inertia -->
-    <!-- These make use of xacro's mathematical functionality -->
-    <xacro:macro name="inertial_sphere" params="mass radius *origin">
-        <inertial>
+<?xml version="1.0" ?>
+<robot name="swerve" xmlns:xacro="http://www.ros.org/wiki/xacro" >
+    <!--
+        A macro to create a wheel link and the joint for the wheel
+        Parameters:
+        - name: Name of the wheel, e.g. left_rear
+        - mass: Mass of the wheel in kilogram
+        - radius: Radius of the wheel in meters
+        - width: Width of the wheel in meters
+        - offset: The distance between the wheel and the steering plate above the wheel. In meters.
+    -->
+    <xacro:macro name="wheel_assembly" params="name mass radius width offset">
+        <joint name="joint_wheel_${name}" type="continuous">
+            <origin rpy="0 0 0" xyz="0 0 ${-1 * (radius + offset)}"/>
+            <parent link="link_steering_${name}"/>
+            <child link="link_wheel_${name}"/>
+            <axis xyz="0.0 1.0 0.0"/>
+        </joint>
+        <link name="link_wheel_${name}">
+            <inertial>
+                <origin xyz="0 0 0" rpy="${PI/2} 0 0" />
+                <mass value="${mass}"/>
+                <inertia
+                    ixx="${(mass/12) * (3*radius*radius + width*width)}"
+                    ixy="0"
+                    ixz="0"
+                    iyy="${(mass/12) * (3*radius*radius + width*width)}"
+                    iyz="0"
+                    izz="${(mass/2) * (radius*radius)}"/>
+            </inertial>
+            <visual>
+                <origin rpy="${PI/2} 0 0" xyz="0 0 0"/>
+                <geometry>
+                    <cylinder length="${width}" radius="${radius}" />
+                </geometry>
+                <material name="black"/>
+            </visual>
+            <collision>
+                <origin rpy="${PI/2} 0 0" xyz="0 0 0"/>
+                <geometry>
+                    <cylinder length="${width}" radius="${radius}" />
+                </geometry>
+            </collision>
+        </link>
+    </xacro:macro>
+    <!--
+        A macro to create a steering link and the joint for the steering unit
+        Parameters:
+        - name: Name of the steering unit, e.g. left_rear
+        - mass: Mass of the steering unit in kilogram
+        - chassis_length: The length of the chassis
+        - chassis_width: The width of the chassis
+        - chassis_height: The height of the chassis
+        - steering_radius: Radius of the steering unit in meters
+        - wheel_radius: Radius of the wheel in meters
+        - thickness: Thickness of the steering unit
+        - offset: The distance between the wheel and the steering plate above the wheel. In meters.
+        - x_reflect: Direction multiplier for X offsets. Either 1 or -1
+        - y_reflect: Direction multiplier for Y offsets. Either 1 or -1
+    -->
+    <xacro:macro name="steering_assembly" params="name parent_link mass chassis_length chassis_width chassis_height steering_radius thickness wheel_radius offset x_reflect y_reflect">
+        <joint name="joint_steering_${name}" type="continuous">
+            <origin rpy="0 0 0" xyz="${x_reflect * (0.5 * chassis_length - steering_radius)} ${y_reflect * (0.5 * chassis_width + steering_radius)} ${0.5 * chassis_height - 0.5 * thickness}"/>
+            <!-- <parent link="chassis_link"/> -->
+            <parent link="${parent_link}"/>
+            <child link="link_steering_${name}"/>
+            <axis xyz="0.0 0.0 1.0"/>
+        </joint>
+        <link name="link_steering_${name}">
+            <inertial>
+                <origin xyz="0 0 0" rpy="0 0 0" />
+                <mass value="${mass}"/>
+                <inertia
+                    ixx="${(mass/12) * (3*steering_radius*steering_radius + thickness*thickness)}"
+                    ixy="0"
+                    ixz="0"
+                    iyy="${(mass/12) * (3*steering_radius*steering_radius + thickness*thickness)}"
+                    iyz="0"
+                    izz="${(mass/2) * (steering_radius*steering_radius)}"/>
+            </inertial>
+            <visual>
+                <origin rpy="0 0 0" xyz="0 0 0"/>
+                <geometry>
+                    <cylinder length="${thickness}" radius="${steering_radius}" />
+                </geometry>
+                <material name="blue"/>
+            </visual>
+            <collision>
+                <origin rpy="0 0 0" xyz="0 0 0"/>
+                <geometry>
+                    <cylinder length="${thickness}" radius="${steering_radius}" />
+                </geometry>
+            </collision>
+            <visual>
+                <origin rpy="0 0 0" xyz="0 ${y_reflect * wheel_radius} ${-1 * 0.5 * (thickness + wheel_radius + 2 * offset)}"/>
+                <geometry>
+                    <box size="${wheel_radius} 0.01 ${wheel_radius + 2 * offset}" />
+                </geometry>
+                <material name="blue"/>
+            </visual>
+            <collision>
+                <origin rpy="0 0 0" xyz="0 ${y_reflect * wheel_radius} ${-1 * 0.5 * (thickness + wheel_radius + 2 * offset)}"/>
+                <geometry>
+                    <box size="${wheel_radius} 0.01 ${wheel_radius + 2 * offset}" />
+                </geometry>
+            </collision>
+        </link>
+    </xacro:macro>
+    <!--
+        A macro to create a wheel link and the joint for the wheel
+        Parameters:
+        - name: Name of the wheel, e.g. left_rear
+        - chassis_length: The length of the chassis
+        - chassis_width: The width of the chassis
+        - chassis_height: The height of the chassis
+        - wheel_mass: Mass of the wheel in kilogram
+        - wheel_radius: Radius of the wheel in meters
+        - wheel_width: Width of the wheel in meters
+        - offset: The distance between the wheel and the steering plate above the wheel. In meters.
+        - x_reflect: Direction multiplier for X offsets. Either 1 or -1
+        - y_reflect: Direction multiplier for Y offsets. Either 1 or -1
+    -->
+    <xacro:macro name="drive_module_assembly" params="name parent_link chassis_length chassis_width chassis_height wheel_mass wheel_radius wheel_width steering_mass steering_radius steering_thickness offset x_reflect y_reflect">
+        <xacro:steering_assembly
+            parent_link="${parent_link}"
+            name="${name}"
+            mass="${steering_mass}"
+            chassis_length="${chassis_length}"
+            chassis_width="${chassis_width}"
+            chassis_height="${chassis_height}"
+            steering_radius="${steering_radius}"
+            thickness="${steering_thickness}"
+            wheel_radius="${wheel_radius}"
+            offset="${offset}"
+            x_reflect="${x_reflect}"
+            y_reflect="${y_reflect}"/>
+        <xacro:wheel_assembly
+            name="${name}"
+            mass="${wheel_mass}"
+            radius="${wheel_radius}"
+            width="${wheel_width}"
+            offset="${offset + 0.5 * steering_thickness}"/>
+    </xacro:macro>
+    <!-- CONTROLLERS -->
+    <xacro:macro name="steering_module_controller" params="name">
+        <joint name="joint_steering_${name}">
+            <command_interface name="position">
+                <param name="min">-${2 * PI}</param>
+                <param name="max">${2 * PI}</param>
+            </command_interface>
+            <state_interface name="position"/>
+            <state_interface name="velocity"/>
+            <!-- <state_interface name="acceleration"/> -->
+        </joint>
+        <joint name="joint_wheel_${name}">
+            <command_interface name="velocity">
+                <param name="min">-1</param>
+                <param name="max">1</param>
+            </command_interface>
+            <state_interface name="position"/>
+            <state_interface name="velocity"/>
+            <!-- <state_interface name="acceleration"/> -->
+        </joint>
+    </xacro:macro>
+    <!-- SENSORS -->
+    <!-- IMU sensor -->
+    <xacro:macro name="sensor_imu" params="name parent_link *origin">
+        <xacro:property name="mass"     value="0.01"/>
+        <xacro:property name="length_x" value="0.01" />
+        <xacro:property name="length_y" value="0.01" />
+        <xacro:property name="length_z" value="0.01" />
+        <xacro:property name="collision_x_offset" value="0.005" />
+        <xacro:property name="collision_y_offset" value="0.005" />
+        <xacro:property name="collision_z_offset" value="${0.5 * length_z}" />
+        <joint name="joint_body_to_sensor_imu_${name}" type="fixed">
             <xacro:insert_block name="origin"/>
-            <mass value="${mass}" />
-            <inertia ixx="${(2/5) * mass * (radius*radius)}" ixy="0.0" ixz="0.0"
-                    iyy="${(2/5) * mass * (radius*radius)}" iyz="0.0"
-                    izz="${(2/5) * mass * (radius*radius)}" />
-        </inertial>
-    </xacro:macro>
-    <xacro:macro name="inertial_box" params="mass x y z *origin">
-        <inertial>
-            <xacro:insert_block name="origin"/>
-            <mass value="${mass}" />
-            <inertia ixx="${(1/12) * mass * (y*y+z*z)}" ixy="0.0" ixz="0.0"
-                    iyy="${(1/12) * mass * (x*x+z*z)}" iyz="0.0"
-                    izz="${(1/12) * mass * (x*x+y*y)}" />
-        </inertial>
-    </xacro:macro>
-    <xacro:macro name="inertial_cylinder" params="mass length radius *origin">
-        <inertial>
-            <xacro:insert_block name="origin"/>
-            <mass value="${mass}" />
-            <inertia ixx="${(1/12) * mass * (3*radius*radius + length*length)}" ixy="0.0" ixz="0.0"
-                    iyy="${(1/12) * mass * (3*radius*radius + length*length)}" iyz="0.0"
-                    izz="${(1/2) * mass * (radius*radius)}"/>
-        </inertial>
+            <parent link="${parent_link}"/>
+            <child link="link_sensor_imu_${name}"/>
+        </joint>
+        <link name="link_sensor_imu_${name}">
+            <visual>
+                <origin xyz="${collision_x_offset} ${collision_y_offset} ${collision_z_offset}"/>
+                <geometry>
+                    <box size="${length_x} ${length_y} ${length_z}"/>
+                </geometry>
+            </visual>
+            <collision>
+                <origin xyz="${collision_x_offset} ${collision_y_offset} ${collision_z_offset}"/>
+                <geometry>
+                    <box size="${length_x} ${length_y} ${length_z}"/>
+                </geometry>
+            </collision>
+            <inertial>
+                <mass value="${mass}" />
+                <xacro:insert_block name="origin"/>
+                <inertia
+                    ixx="${(1/12) * mass * (length_y*length_y + length_z*length_z)}"
+                    ixy="0.0"
+                    ixz="0.0"
+                    iyy="${(1/12) * mass * (length_x*length_x + length_z*length_z)}"
+                    iyz="0.0"
+                    izz="${(1/12) * mass * (length_x*length_x + length_y*length_y)}" />
+            </inertial>
+        </link>
+    </xacro:macro>
+    <!-- Lidar sensor -->
+    <xacro:macro name="sensor_lidar" params="name parent_link chassis_top_relative_height">
+        <xacro:property name="mass"     value="0.17"/>
+        <xacro:property name="length_x" value="0.071" />
+        <xacro:property name="length_y" value="0.10" />
+        <xacro:property name="length_z" value="0.06" />
+        <xacro:property name="collision_x_offset" value="0" />
+        <xacro:property name="collision_y_offset" value="0" />
+        <xacro:property name="collision_z_offset" value="${chassis_top_relative_height}" />
+        <joint name="joint_body_to_sensor_lidar_${name}" type="fixed">
+            <parent link="${parent_link}"/>
+            <child link="link_sensor_lidar_${name}"/>
+            <origin rpy="0 0 0" xyz="${collision_x_offset} ${collision_y_offset} ${collision_z_offset}"/>
+        </joint>
+        <link name="link_sensor_lidar_${name}">
+            <visual>
+                <origin rpy="0 0 0" xyz="0.0 0 ${0.5 * length_z}"/>
+                <geometry>
+                    <box size="${length_x} ${length_y} ${length_z}"/>
+                </geometry>
+            </visual>
+            <collision>
+                <origin rpy="0 0 0" xyz="0.0 0 ${0.5 * length_z}"/>
+                <geometry>
+                    <box size="${length_x} ${length_y} ${length_z}"/>
+                </geometry>
+            </collision>
+            <inertial>
+                <mass value="${mass}" />
+                <origin rpy="0 0 0" xyz="0.0 0 ${0.5 * length_z}"/>
+                <inertia
+                    ixx="${(1/12) * mass * (length_y*length_y + length_z*length_z)}"
+                    ixy="0.0"
+                    ixz="0.0"
+                    iyy="${(1/12) * mass * (length_x*length_x + length_z*length_z)}"
+                    iyz="0.0"
+                    izz="${(1/12) * mass * (length_x*length_x + length_y*length_y)}" />
+            </inertial>
+        </link>
     </xacro:macro>
 </robot>

File: src/swerve_drive_description/urdf/materials.xacro (robot description, xacro)
@@ -1,12 +1,18 @@
 <?xml version="1.0" ?>
-<robot name="amr" xmlns:xacro="http://www.ros.org/wiki/xacro" >
-<material name="silver">
-  <color rgba="0.700 0.700 0.700 1.000"/>
-</material>
-<material name="berry" >
-  <color rgba="0.6 0.058823529411764705 0.29411764705882354 1.0" />
-</material>
-<material name="red" >
-  <color rgba="1 0.0 0.0 1.0" />
-</material>
+<robot name="swerve" xmlns:xacro="http://www.ros.org/wiki/xacro" >
+    <material name="black">
+        <color rgba="0.01 0.01 0.01 1.000"/>
+    </material>
+    <material name="silver">
+        <color rgba="0.700 0.700 0.700 1.000"/>
+    </material>
+    <material name="gray">
+        <color rgba="0.250 0.250 0.250 1.000"/>
+    </material>
+    <material name="blue">
+        <color rgba="0.000 0.000 0.700 1.000"/>
+    </material>
+    <material name="orange">
+        <color rgba="1.000 0.624 0.000 1.000"/>
+    </material>
 </robot>
